File: tinyswr.sch (KiCad schematic (older format))
At the start: 15 parts, among them J1 ANT, J2 RIG

Commit message: fixed missing gnd connection and other bugs
Parts:
- removed R2: 1k, lib_fp:Potentiometer_Trimmer_Bourns_3314G, symbol RTRIM
- added R2: 1k, lib_fp:Potentiometer_Trimmer_Bourns_3314G, symbol POT_TRIM
Connections:
- net GND: now also D3.2 (A), R3.2, R4.2, R5.2, RF1.1 (K), SWR3.1 (K)
- net at D1.2 (A), D2.1 (K), L1.3 (2-1)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: now also R2.2, R2.3
- net at R1.2: now also R2.1
Changed lines of the file:
@@
 Sheet 1 1
 Title "TinySWR"
-Date ""
+Date "2017/10/24"
 Rev "1.2"
 Comp "Martin Hepp, DK3IT"
@@
 $EndComp
 $Comp
-L RTRIM R2
-U 1 1 5974AD26
-P 4500 2850
-F 0 "R2" V 4600 2750 50  0000 L CNN
-F 1 "1k" V 4400 2825 50  0000 L CNN
-F 2 "lib_fp:Potentiometer_Trimmer_Bourns_3314G" V 4430 2850 50  0001 C CNN
-F 3 "http://www.mouser.com/ds/2/54/314-776736.pdf" H 4500 2850 50  0001 C CNN
-F 4 "n/a" H 4500 2850 60  0001 C CNN "Datasheet URI"
-F 5 "Bourns" V 4500 2850 60  0001 C CNN "MFN"
-F 6 "3314G-1-102E" V 4500 2850 60  0001 C CNN "MFP"
-	1    4500 2850
-	1    0    0    -1
-$EndComp
-$Comp
 L FT23-43 L1
 U 1 1 59767ABF
@@
 L GND #PWR01
 U 1 1 5977B389
-P 3700 2600
-F 0 "#PWR01" H 3700 2350 50  0001 C CNN
-F 1 "GND" H 3700 2450 50  0000 C CNN
-F 2 "" H 3700 2600 50  0001 C CNN
-F 3 "" H 3700 2600 50  0001 C CNN
-	1    3700 2600
+P 3700 2950
+F 0 "#PWR01" H 3700 2700 50  0001 C CNN
+F 1 "GND" H 3700 2800 50  0000 C CNN
+F 2 "" H 3700 2950 50  0001 C CNN
+F 3 "" H 3700 2950 50  0001 C CNN
+	1    3700 2950
 	1    0    0    -1
 $EndComp
@@
 L GND #PWR02
 U 1 1 59A56D88
-P 6900 2600
-F 0 "#PWR02" H 6900 2350 50  0001 C CNN
-F 1 "GND" H 6900 2450 50  0000 C CNN
-F 2 "" H 6900 2600 50  0001 C CNN
-F 3 "" H 6900 2600 50  0001 C CNN
-	1    6900 2600
+P 6900 2950
+F 0 "#PWR02" H 6900 2700 50  0001 C CNN
+F 1 "GND" H 6900 2800 50  0000 C CNN
+F 2 "" H 6900 2950 50  0001 C CNN
+F 3 "" H 6900 2950 50  0001 C CNN
+	1    6900 2950
 	1    0    0    -1
 $EndComp
@@
 Connection ~ 5200 3350
 Wire Wire Line
-	4400 3000 4500 3000
-Wire Wire Line
 	4500 3350 5500 3350
 Connection ~ 4900 3350
 Wire Wire Line
-	4150 2500 4150 4300
-Wire Wire Line
 	3850 2400 5000 2400
 Wire Wire Line
 	6750 2400 5300 2400
 Connection ~ 4500 2400
-Wire Wire Line
-	4400 2950 4400 3000
-Connection ~ 4500 3000
 Wire Wire Line
 	4500 3000 4500 3700
@@
 Connection ~ 5200 4300
 Connection ~ 5500 4300
-Connection ~ 4400 2950
 Connection ~ 4500 4300
 Connection ~ 4500 3350
@@
 Wire Wire Line
 	5300 2500 6050 2500
-Wire Wire Line
-	6900 2500 6700 2500
-Wire Wire Line
-	6700 2500 6700 4300
-Connection ~ 6900 2500
 Connection ~ 11000 -3350
 Connection ~ 5200 3650
@@
 	-1   0    0    -1
 $EndComp
-Wire Wire Line
-	3700 2500 4150 2500
-Connection ~ 3700 2500
 Text Notes 3525 4900 0    60   ~ 0
 The choice of LEDs is critical. The following types work well in my tests:\nSWR1-3: KINGBRIGHT L-934LID (Reichelt: LED 3MM 2MA RT), Forward Voltage typ 1.7, max 2.0\nRF1: KINGBRIGHT L-934LYD (Reichelt: LED 3MM 2MA GE) Forward Voltage typ 1.8, max 2.1 V\nD1: OSRAM OPTO LS M67K-H2L1-1-Z (Reichelt: LS M67K), Forward Voltage min: 1.7, max 2.2, typ 1.8 V
+Wire Wire Line
+	3700 2600 3700 2950
+Wire Wire Line
+	4150 4300 4150 2775
+Wire Wire Line
+	4150 2775 3700 2775
+Connection ~ 3700 2775
+Wire Wire Line
+	6900 2600 6900 2950
+Wire Wire Line
+	6700 4300 6700 2725
+Wire Wire Line
+	6700 2725 6900 2725
+Connection ~ 6900 2725
+$Comp
+L POT_TRIM R2
+U 1 1 59EF8800
+P 4500 2850
+F 0 "R2" V 4325 2850 50  0000 C CNN
+F 1 "1k" V 4400 2850 50  0000 C CNN
+F 2 "lib_fp:Potentiometer_Trimmer_Bourns_3314G" H 4500 2850 50  0001 C CNN
+F 3 "http://www.mouser.com/ds/2/54/314-776736.pdf" H 4500 2850 50  0001 C CNN
+F 4 "Bourns" H 4500 2850 60  0001 C CNN "MFN"
+F 5 "3314G-1-102E" H 4500 2850 60  0001 C CNN "MPN"
+F 6 "652-3314G-1-102E" H 4500 2850 60  0001 C CNN "Mouser Part Number"
+F 7 "https://www.mouser.de/ProductDetail/Bourns/3314G-1-102E/" H 4500 2850 60  0001 C CNN "Mouser Part Link"
+F 8 "Reichelt" H 4500 2850 60  0001 C CNN "Alternative Source Name"
+F 9 "23B-1,0K" H 4500 2850 60  0001 C CNN "Alternative Source Part Number"
+F 10 "1k" H 4500 2850 60  0001 C CNN "Characteristics"
+F 11 "n/a" H 4500 2850 60  0001 C CNN "Description"
+F 12 "n/a" H 4500 2850 60  0001 C CNN "Package ID"
+F 13 "ANY" H 4500 2850 60  0001 C CNN "Source"
+F 14 "Y" H 4500 2850 60  0001 C CNN "Critical"
+F 15 "n/a" H 4500 2850 60  0001 C CNN "Notes"
+F 16 "n/a" H 4500 2850 60  0001 C CNN "Design Decision URI"
+F 17 "Value" H 4500 2850 60  0001 C CNN "Fieldname"
+	1    4500 2850
+	1    0    0    -1
+$EndComp
+Wire Wire Line
+	4650 2850 4650 3025
+Wire Wire Line
+	4650 3025 4500 3025
+Connection ~ 4500 3025
 $EndSCHEMATC
